File: esp32s2-nixiehost/esp32s2-nixiehost.kicad_pcb (KiCad board)
At the start: 2 copper layers, 16.6 x 1.8 mm, 50 parts, among them J1 USB_C_Receptacle_USB2.0, J10 OUTPUTSLOTS3, J2 PGM, J3 OUTPUTPINS0, J4 OUTPUTPINS1, J5 OUTPUTPINS2, J6 OUTPUTPINS3, J7 OUTPUTSLOTS0, J8 OUTPUTSLOTS1, J9 OUTPUTSLOTS2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

Commit message: Bump to rel ver
Parts:
- added J11: OUTPUTPINS5, Connector_PinSocket_2.54mm:PinSocket_2x05_P2.54mm_Vertical_SMD, F.Cu at (169.0, 111.0)
- added J12: OUTPUTPINS4, Connector_PinSocket_2.54mm:PinSocket_2x05_P2.54mm_Vertical_SMD, F.Cu at (146.0, 111.0)
- added J13: OUTPUTSLOTS5, nixiehostslot:nixiehostslot, F.Cu at (169.0, 119.0)
- added J14: OUTPUTSLOTS4, nixiehostslot:nixiehostslot, F.Cu at (146.0, 119.0)
- added J15: ~, MountingHole:MountingHole_3.5mm_Pad, F.Cu at (48.0, 92.0)
- added J16: ~, MountingHole:MountingHole_3.5mm_Pad, F.Cu at (177.0, 92.0)
- added J17: ~, MountingHole:MountingHole_3.5mm_Pad, F.Cu at (177.0, 141.0)
- added J18: ~, MountingHole:MountingHole_3.5mm_Pad, F.Cu at (48.0, 141.0)
- added R11: 10k, Resistor_SMD:R_0402_1005Metric, F.Cu at (142.9, 105.0)
- added R12: 10k, Resistor_SMD:R_0402_1005Metric, F.Cu at (166.0, 104.8)
- moved T6 21.0 mm to (151.0, 140.8)
- moved A1 20.5 mm to (72.1, 89.3), turned to 90 degrees
- moved T5 19.0 mm to (135.0, 140.9)
- moved T4 18.0 mm to (120.0, 140.9)
- moved T3 16.0 mm to (104.0, 141.0)
- moved T2 14.0 mm to (88.0, 140.9)
- moved T1 12.0 mm to (72.0, 141.0)
- moved D1 9.13 mm to (105.7, 97.5), turned to 0 degrees
- moved C7 4.06 mm to (95.2, 97.5), turned to 90 degrees
- moved C1 2.52 mm to (75.2, 102.2)
- moved C2 2.52 mm to (78.3, 102.2)
- moved L1 2.52 mm to (76.8, 102.8)
- moved R9 1.23 mm to (114.3, 96.4)
- moved D2 1.21 mm to (109.7, 100.9)
- moved R10 1.11 mm to (109.4, 96.4)
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Connections:
- U1 pad 19: GND -> unconnected-(U1-Pad19)
Routing:
- net GND: track 0.00 -> 295.2 mm, vias 0 -> 70
- net VBUS: track 0.00 -> 231.1 mm, vias 0 -> 23
- net VDD: track 0.00 -> 166.9 mm, vias 0 -> 11
- net LEDCTL5: track 0.00 -> 94.9 mm
- net Net-(T6-Pad1): track 0.00 -> 88.8 mm
- net Net-(T5-Pad1): track 0.00 -> 73.9 mm
- net LEDCTL4: track 0.00 -> 71.9 mm
- net Net-(T4-Pad1): track 0.00 -> 60.4 mm
- net LEDCTL0: track 0.00 -> 56.4 mm, vias 0 -> 2
- net LEDCTL3: track 0.00 -> 48.8 mm
- net Net-(T1-Pad1): track 0.00 -> 47.8 mm
- net Net-(T3-Pad1): track 0.00 -> 47.5 mm
- net Net-(T2-Pad1): track 0.00 -> 41.0 mm
- net GPIO0: track 0.00 -> 33.9 mm, vias 0 -> 4
- net LEDCTL1: track 0.00 -> 33.3 mm, vias 0 -> 2
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- added copper zone on B.Cu, net GND
- added copper zone on F.Cu, net GND
Other:
- board size 16.6 x 1.8 mm -> 139 x 59 mm
- board text added: "*"
- board text added: "esp32s2-nixiehost rev -"
- board text removed: "TODO: CHECK ORIENTATION (Forwards backwards) The connectors CANNOT be on TUBE side. TOUCH MUST BE IN FRONT"
