File: esp32s2-nixiehost/esp32s2-nixiehost.kicad_sch (KiCad schematic)
At the start: 50 parts, among them J1 USB_C_Receptacle_USB2.0, J10 OUTPUTSLOTS3, J2 PGM, J3 OUTPUTPINS0, J4 OUTPUTPINS1, J5 OUTPUTPINS2, J6 OUTPUTPINS3, J7 OUTPUTSLOTS0, J8 OUTPUTSLOTS1, J9 OUTPUTSLOTS2, SW1 TS-1187A-B-A-B, T1 TOUCH, T2 TOUCH, T3 TOUCH, T4 TOUCH, T5 TOUCH, T6 TOUCH, U1 ESP32-S2, U2 ME6206A36M3G, Y1 40MHz, Y2 32.786k

Commit message: Bump to rel ver
Parts:
- added J11: OUTPUTPINS5, Connector_PinSocket_2.54mm:PinSocket_2x05_P2.54mm_Vertical_SMD, symbol Connector_Generic:Conn_02x05_Odd_Even
- added J12: OUTPUTPINS4, Connector_PinSocket_2.54mm:PinSocket_2x05_P2.54mm_Vertical_SMD, symbol Connector_Generic:Conn_02x05_Odd_Even
- added J13: OUTPUTSLOTS5, nixiehostslot:nixiehostslot, symbol Connector_Generic:Conn_01x03
- added J14: OUTPUTSLOTS4, nixiehostslot:nixiehostslot, symbol Connector_Generic:Conn_01x03
- added J15, J16, J17, J18: ~, MountingHole:MountingHole_3.5mm_Pad, symbol Connector_Generic:Conn_01x01
- added R11, R12: 10k, Resistor_SMD:R_0402_1005Metric, symbol Device:R
- D2: LCSC C5199107 -> C115330
- J3, J4, J5, J6: LCSC C920845 -> C843271
Connections:
- net GND: now also J11.1 (Pin_1), J11.10 (Pin_10), J11.2 (Pin_2), J11.9 (Pin_9), J12.1 (Pin_1), J12.10 (Pin_10), J12.2 (Pin_2), J12.9 (Pin_9), J13.1 (Pin_1), J14.1 (Pin_1), J15.1 (Pin_1), J16.1 (Pin_1), J17.1 (Pin_1), J18.1 (Pin_1); no longer U1.19 (GPIO14)
- net LEDCTL4: now also J12.3 (Pin_3), J12.8 (Pin_8), J14.3 (Pin_3), R11.1
- net LEDCTL5: now also J11.3 (Pin_3), J11.8 (Pin_8), J13.3 (Pin_3), R12.1
- net VBUS: now also J11.5 (Pin_5), J11.6 (Pin_6), J12.5 (Pin_5), J12.6 (Pin_6), J13.2 (Pin_2), J14.2 (Pin_2)
- net VDD: now also R11.2, R12.2
Other:
- moved on the sheet: J10, J3, J4, J5, J6, J7, J8, J9
